File: linearlight/linearlight.kicad_pcb (KiCad board)
At the start: 2 copper layers, 141 x 59.7 mm, 82 parts, among them J1 Screw_Terminal, J2 Conn_01x04_Pin, J3 Conn_01x19_Socket, J4 Conn_01x19_Socket, J5 Conn_01x04_Pin, J6 Conn_01x08_Socket, Q1 FQP30N06, Q2 FQP30N06, Q3 FQP30N06, Q4 FQP30N06, Q5 2N3904, Q6 2N3904, Q7 2N3904, Q8 2N3904, U1 TLV5620CN, U2 ESP32 DevKitC, U3 MC33204, U4 LM4040LP-2.5, U5 TLV5620CN, U6 L7805

Commit message: Add usage text
Changed lines of the file:
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@@
     (property "ki_keywords" "cap capacitor")
     (attr through_hole)
-    (fp_text reference "C1" (at 1.25 -2.5) (layer "F.SilkS")
+    (fp_text reference "C1" (at 3.917 2.413) (layer "F.SilkS")
         (effects (font (size 1 1) (thickness 0.15)))
     )
