File: linearlight/linearlight.kicad_sch (KiCad schematic)
At the start: 72 parts, among them J1 Screw_Terminal, J2 Conn_01x04_Pin, J3 Conn_01x19_Socket, J4 Conn_01x19_Socket, J5 Conn_01x04_Pin, Q1 FQP30N06, Q2 FQP30N06, Q3 FQP30N06, Q4 FQP30N06, Q5 2N3904, Q6 2N3904, Q7 2N3904, Q8 2N3904, U1 TLV5620CN, U2 ESP32 DevKitC, U3 MC33204, U4 LM4040LP-2.5

Commit message: Updates including 2nd DAC for nonlinear response.
Parts:
- removed C9: 2200uF, Capacitor_THT:CP_Radial_D13.0mm_P5.00mm, symbol Device:C_Polarized
- removed F1: Fuse, Fuse:01530008, symbol Device:Fuse
- removed H4: MountingHole, MountingHole:MountingHole_3.2mm_M3, symbol Mechanical:MountingHole
- removed R16, R17, R18, R19: 100k, Resistor_THT:R_Axial_DIN0204_L3.6mm_D1.6mm_P7.62mm_Horizontal, symbol Device:R
- added C10: 100u, Capacitor_THT:CP_Radial_D6.3mm_P2.50mm, symbol Device:C_Polarized
- added C9: 1u, Capacitor_THT:C_Disc_D5.0mm_W2.5mm_P2.50mm, symbol Device:C
- added D2, D3, D4, D5: 1N4148, Diode_THT:D_DO-35_SOD27_P7.62mm_Horizontal, symbol Diode:1N4148
- added F2: Fuse, Fuse:01530008, symbol Device:Fuse
- added U5: TLV5620CN, Package_DIP:DIP-14_W7.62mm_Socket, symbol Analog_DAC_TI:TLV5620CN
- C7: value 100u -> 2200uF; footprint Capacitor_THT:CP_Radial_D6.3mm_P2.50mm -> Capacitor_THT:CP_Radial_D13.0mm_P5.00mm
- H1, H2, H3: value MountingHole -> ~
- HS1, HS2, HS3, HS4: value Heatsink -> ~
- R12, R15, R2, R9: footprint Resistor_THT:RES_WLAR100FET -> Resistor_THT:R_Axial_DIN0207_L6.3mm_D2.5mm_P10.16mm_Horizontal
- R28: footprint Resistor_THT:R_Axial_DIN0207_L6.3mm_D2.5mm_P10.16mm_Horizontal -> Resistor_THT:R_Axial_DIN0204_L3.6mm_D1.6mm_P7.62mm_Horizontal
- R4: value 4.7k -> 10k
- U4: footprint Package_TO_SOT_THT:TO-92_Inline -> Package_TO_SOT_THT:TO-92_Inline_Wide
Connections:
- net +12V: now also C7.1, F2.2
- net +5V: now also C10.1, C9.1, U5.14 (VDD); no longer C7.1
- net GND: now also C10.2, C9.2, U5.1 (GND)
- net at U3.2 (IN-): now also C1.2, R6.1, D2.1 (K); no longer U1.11 (DACB)
- net at J3.13 (Pin_13), U2.7 (GPIO32,ADC1_CH4): now also R30.1; no longer R31.1
- net at C6.2, R14.1: now also U3.13 (IN-), D5.1 (K); no longer U3.12 (IN+)
- net at U1.10 (DACC): now also U3.10 (IN+); no longer U3.13 (IN-)
- net at J3.12 (Pin_12), U2.8 (GPIO33,ADC1_CH5): now also R31.1; no longer R32.1
- net at C4.2, R8.1: now also U3.6 (IN-), D3.1 (K); no longer U3.5 (IN+)
- net at U1.12 (DACA): now also U3.3 (IN+); no longer U3.6 (IN-)
- net at J3.17 (Pin_17), R4.2, R5.1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: now also U5.2 (REFA), U5.3 (REFB), U5.4 (REFC), U5.5 (REFD); no longer U1.2 (REFA), U1.3 (REFB), U1.4 (REFC), U1.5 (REFD)
- net at C5.2, R11.1: now also U3.9 (IN-), D4.1 (K); no longer U3.10 (IN+)
- net at J3.9 (Pin_9), U1.6 (DATA), U2.11 (GPIO27,ADC2_CH7): now also U5.6 (DATA)
- net at J3.10 (Pin_10), U1.7 (CLK), U2.10 (GPIO26,ADC2_CH9,DAC_2): now also U5.7 (CLK)
- net at U1.9 (DACD): now also U3.12 (IN+); no longer U3.9 (IN-)
- net at J4.3 (Pin_3), U2.36 (GPIO22): now also J5.4 (Pin_4); no longer J5.3 (Pin_3)
- net at J4.6 (Pin_6), U2.33 (GPIO21): now also J5.3 (Pin_3); no longer J5.4 (Pin_4)
- net at J3.15 (Pin_15), U2.5 (GPIO34,ADC1_CH6,VDET_1): now also R29.1; no longer R30.1
- net at J4.13 (Pin_13), U2.26 (GPIO4,ADC2_CH0): now also D2.2 (A)
- net at J4.14 (Pin_14), U2.25 (GPIO0,ADC2_CH1): now also D3.2 (A)
- net at J4.15 (Pin_15), U2.24 (GPIO2,ADC2_CH2): now also D4.2 (A)
- net at J4.16 (Pin_16), U2.23 (GPIO15,ADC2_CH3): now also D5.2 (A)
- net at J1.1 (Pin_1): now also F2.1
- net at J3.7 (Pin_7), U2.13 (GPIO12,ADC2_CH5): now also U5.8 (LOAD)
- net at J3.16 (Pin_16), U2.4 (GPIO39,ADC1_CH3,S_VN): no longer R29.1
- net at J3.14 (Pin_14), U2.6 (GPIO35,ADC1_CH7,VDET_2): now also R32.1
- new net: U1.11 (DACB), U3.5 (IN+)
- new net: U1.2 (REFA), U5.12 (DACA)
- new net: U1.3 (REFB), U5.11 (DACB)
- new net: U1.4 (REFC), U5.10 (DACC)
- new net: U1.5 (REFD), U5.9 (DACD)
Other:
- note added: "Tested current with Green channel of 5 metre strip: With 0.15Ω current sense, sense voltage is 0.178mV ~ 1.18A"
- moved on the sheet: C3, C8, D1, J1, J5, R28, R29, R3, R30, R31, R32, R4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

Commit message: PCB layout passes DRC.
Parts:
- added C11, C12, C13, C14, C15: 0.1u, Capacitor_THT:C_Disc_D5.0mm_W2.5mm_P2.50mm, symbol Device:C
- added C17: .1u, Capacitor_THT:C_Disc_D5.0mm_W2.5mm_P2.50mm, symbol Device:C
- added U6: L7805, Package_TO_SOT_THT:TO-220-3_Vertical, symbol Regulator_Linear:L7805
- D1: footprint LED_THT:LED_D5.0mm -> LED_THT:LED_D3.0mm
- HS1, HS2, HS3, HS4: footprint Heatsink:Max48 heatsink -> Heatsink:Max47 heatsink
- R12, R15, R2, R9: value 0.15 -> 0.5; footprint Resistor_THT:R_Axial_DIN0207_L6.3mm_D2.5mm_P10.16mm_Horizontal -> Resistor_THT:R_Axial_DIN0414_L11.9mm_D4.5mm_P5.08mm_Vertical
- R4: value 10k -> 2.2k
Connections:
- net +12V: now also U6.1 (IN)
- net +5V: now also C17.1, U6.3 (OUT)
- net GND: now also C11.1, C12.1, C13.1, C14.1, C15.1, C17.2, U6.2 (GND)
- net at J3.12 (Pin_12), U2.8 (GPIO33,ADC1_CH5): now also R30.1, C12.2; no longer R31.1
- net at Q3.3 (S), R11.2, R12.1: now also R30.2; no longer R31.2
- net at J3.14 (Pin_14), U2.6 (GPIO35,ADC1_CH7,VDET_2): now also R29.1, C11.2; no longer R32.1
- net at Q4.3 (S), R14.2, R15.1: now also R29.2; no longer R32.2
- net at J4.15 (Pin_15), U2.24 (GPIO2,ADC2_CH2): no longer D4.2 (A)
- net at J3.17 (Pin_17), R4.2, R5.1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: now also C15.2
- net at Q1.3 (S), R2.1, R6.2: now also R32.2; no longer R29.2
- net at Q2.2 (D): now also J1.4 (Pin_4); no longer J1.3 (Pin_3)
- net at Q2.3 (S), R8.2, R9.1: now also R31.2; no longer R30.2
- net at Q3.2 (D): now also J1.5 (Pin_5); no longer J1.4 (Pin_4)
- net at J4.8 (Pin_8), U2.31 (GPIO19): now also J5.3 (Pin_3); no longer R26.1
- net at J4.6 (Pin_6), U2.33 (GPIO21): no longer J5.3 (Pin_3)
- net at J4.3 (Pin_3), U2.36 (GPIO22): now also U5.8 (LOAD); no longer J5.4 (Pin_4)
- net at J4.16 (Pin_16), U2.23 (GPIO15,ADC2_CH3): no longer D5.2 (A)
- net at J4.2 (Pin_2), U2.37 (GPIO23): now also U5.13 (LDAC); no longer R21.1
- net at J3.13 (Pin_13), U2.7 (GPIO32,ADC1_CH4): now also R31.1, C13.2; no longer R30.1
- net at Q4.2 (D): now also J1.3 (Pin_3); no longer J1.5 (Pin_5)
- net at J4.14 (Pin_14), U2.25 (GPIO0,ADC2_CH1): no longer D3.2 (A)
- net at J4.10 (Pin_10), U2.29 (GPIO5): now also D3.2 (A), R24.1; no longer R22.1
- net at J4.13 (Pin_13), U2.26 (GPIO4,ADC2_CH0): now also D4.2 (A), R22.1; no longer D2.2 (A)
- net at J4.4 (Pin_4), U2.35 (GPIO1,U0TXD): now also D2.2 (A), R26.1
- net at J4.5 (Pin_5), U2.34 (GPIO3,U0RXD): now also D5.2 (A), R21.1
- net at J4.9 (Pin_9), U2.30 (GPIO18): now also J5.4 (Pin_4); no longer R24.1
- net at J3.7 (Pin_7), U2.13 (GPIO12,ADC2_CH5): no longer U5.8 (LOAD)
- net at J3.15 (Pin_15), U2.5 (GPIO34,ADC1_CH6,VDET_1): now also R32.1, C14.2; no longer R29.1
Other:
- moved on the sheet: C1, C10, C2, C3, C4, C5, C6, C7, C8, C9, D1, D2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

Commit message: Release candidate 1
Parts:
- added TP_VDAC1: VDAC, TestPoint:TestPoint_THTPad_2.5x2.5mm_Drill1.2mm, symbol Connector:TestPoint
- renumbered TP1 to TP+12, TP4 to TP+2.5, TP2 to TP+5, TP3 to TP_GND1
Connections:
- net at C15.2, J3.17 (Pin_17), R4.2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: now also TP_VDAC1.1
Changed lines of the file:
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@@
   (junction (at 231.14 72.39) (diameter 0) (color 0 0 0 0)
   )
+  (junction (at 44.45 110.49) (diameter 0) (color 0 0 0 0)
+  )
   (junction (at 223.52 135.89) (diameter 0) (color 0 0 0 0)
   )
@@
   (symbol (lib_id "Connector:TestPoint") (at 332.74 99.06 0) (unit 1)
     (in_bom yes) (on_board yes) (dnp no)
-    (property "Reference" "TP1" (at 335.28 94.488 0)
+    (property "Reference" "TP+12" (at 335.28 94.488 0)
       (effects (font (size 1.27 1.27)) (justify left))
     )
@@
       (project "linearlight"
         (path "/9f31f3ef-fa50-46f5-aec7-55370bc57602"
-          (reference "TP1") (unit 1)
+          (reference "TP+12") (unit 1)
         )
       )
@@
   (symbol (lib_id "Connector:TestPoint") (at 346.71 106.68 0) (unit 1)
     (in_bom yes) (on_board yes) (dnp no) (fields_autoplaced)
-    (property "Reference" "TP2" (at 349.25 102.108 0)
+    (property "Reference" "TP+5" (at 349.25 102.108 0)
       (effects (font (size 1.27 1.27)) (justify left))
     )
@@
       (project "linearlight"
         (path "/9f31f3ef-fa50-46f5-aec7-55370bc57602"
-          (reference "TP2") (unit 1)
+          (reference "TP+5") (unit 1)
         )
       )
@@
     )
   )
+  (symbol (lib_id "Connector:TestPoint") (at 44.45 110.49 0) (unit 1)
+    (in_bom yes) (on_board yes) (dnp no) (fields_autoplaced)
+    (property "Reference" "TP_VDAC1" (at 46.99 105.918 0)
+      (effects (font (size 1.27 1.27)) (justify left))
+    )
+    (property "Value" "VDAC" (at 46.99 108.458 0)
+      (effects (font (size 1.27 1.27)) (justify left))
+    )
+    (property "Footprint" "TestPoint:TestPoint_THTPad_2.5x2.5mm_Drill1.2mm" (at 49.53 110.49 0)
+      (effects (font (size 1.27 1.27)) hide)
+    )
+    (property "Datasheet" "~" (at 49.53 110.49 0)
+      (effects (font (size 1.27 1.27)) hide)
+    )
+    (pin "1")
+    (instances
+      (project "linearlight"
+        (path "/9f31f3ef-fa50-46f5-aec7-55370bc57602"
+          (reference "TP_VDAC1") (unit 1)
+        )
+      )
+    )
+  )
   (symbol (lib_id "Device:R") (at 219.71 77.47 90) (unit 1)
     (in_bom yes) (on_board yes) (dnp no) (fields_autoplaced)
@@
   (symbol (lib_id "Connector:TestPoint") (at 332.74 104.14 0) (unit 1)
     (in_bom yes) (on_board yes) (dnp no)
-    (property "Reference" "TP3" (at 335.28 99.568 0)
+    (property "Reference" "TP_GND1" (at 335.28 99.568 0)
       (effects (font (size 1.27 1.27)) (justify left))
     )
@@
       (project "linearlight"
         (path "/9f31f3ef-fa50-46f5-aec7-55370bc57602"
-          (reference "TP3") (unit 1)
+          (reference "TP_GND1") (unit 1)
         )
       )
@@
   (symbol (lib_id "Connector:TestPoint") (at 38.1 132.08 0) (unit 1)
     (in_bom yes) (on_board yes) (dnp no) (fields_autoplaced)
-    (property "Reference" "TP4" (at 40.64 127.508 0)
+    (property "Reference" "TP+2.5" (at 40.64 127.508 0)
       (effects (font (size 1.27 1.27)) (justify left))
     )
@@
       (project "linearlight"
         (path "/9f31f3ef-fa50-46f5-aec7-55370bc57602"
-          (reference "TP4") (unit 1)
+          (reference "TP+2.5") (unit 1)
         )
       )

Commit message: Release candidate 2
Connections:
- net at J3.11 (Pin_11), U2.9 (GPIO25,ADC1_CH8,DAC_1): now also U1.8 (LOAD); no longer U1.13 (LDAC)
- net at U1.6 (DATA), U5.6 (DATA): now also J3.8 (Pin_8), U2.12 (GPIO14,ADC2_CH6); no longer J3.9 (Pin_9), U2.11 (GPIO27,ADC2_CH7)
- net at J3.10 (Pin_10), U2.10 (GPIO26,ADC2_CH9,DAC_2): now also U1.13 (LDAC); no longer U1.7 (CLK), U5.7 (CLK)
- new net: J3.9 (Pin_9), U1.7 (CLK), U2.11 (GPIO27,ADC2_CH7), U5.7 (CLK)
Other:
- note added: "BLUE"
- note added: "CONTROL DAC"
- note added: "GREEN"
- note added: "RED"
- note added: "SCALE DAC"
- note added: "WHITE"
